Commit message: Updated Collision models

File: urdf/Paucibot.urdf (robot description, URDF)
Before this commit: robot Paucibot, 15 links, 14 joints
Links:
- link UpperLink: geometry collision cylinder length=0.0055 radius=0.075; visual cylinder length=0.0055 radius=0.075
- link UpperPillar2: mass 0.07 -> 0.001
